File: PCB/keyboard.kicad_sch (KiCad schematic)
At the start: 158 parts, among them SW1 SW_Push, SW10 SW_Push, SW11 SW_Push, SW12 SW_Push, SW13 SW_Push, SW14 SW_Push, SW15 SW_Push, SW16 SW_Push, SW17 SW_Push, SW18 SW_Push, SW19 SW_Push, SW2 SW_Push, SW20 SW_Push, SW21 SW_Push, SW22 SW_Push, SW23 SW_Push, SW24 SW_Push, SW25 SW_Push, SW27 SW_Push, SW28 SW_Push, SW29 SW_Push, SW3 SW_Push, SW30 SW_Push, SW31 SW_Push, SW33 SW_Push, SW34 SW_Push, SW35 SW_Push, SW36 SW_Push, SW37 SW_Push, SW38 SW_Push, SW39 SW_Push, SW4 SW_Push, SW40 SW_Push, SW42 SW_Push, SW43 SW_Push, SW44 SW_Push, SW45 SW_Push, SW46 SW_Push, SW47 SW_Push, SW48 SW_Push, SW49 SW_Push, SW5 SW_Push, SW50 SW_Push, SW51 SW_Push, SW52 SW_Push, SW53 SW_Push, SW54 SW_Push, SW55 SW_Push, SW56 SW_Push, SW58 SW_Push, SW59 SW_Push, SW6 SW_Push, SW61 SW_Push, SW62 SW_Push, SW63 SW_Push, SW64 SW_Push, SW65 SW_Push, SW67 SW_Push, SW68 SW_Push, SW7 SW_Push, SW70 SW_Push, SW71 SW_Push, SW72 SW_Push, SW73 SW_Push, SW74 SW_Push, SW75 SW_Push, SW77 SW_Push, SW78 SW_Push, SW79 SW_Push, SW8 SW_Push, SW81 SW_Push, SW84 SW_Push, SW85 SW_Push, SW87 SW_Push, SW9 SW_Push, SW90 SW_Push

Commit message: feat: new images project and finished pcb
Parts:
- added D59, D63, D64, D65, D68, D69, D70, D71, D72, D73, D74: 1N4148, Diode_THT:D_DO-35_SOD27_P7.62mm_Horizontal, symbol Diode:1N4148
- added SW57, SW60, SW64, SW65, SW66, SW69, SW70, SW71, SW72, SW73, SW74, SW75: SW_Push, PCM_marbastlib-mx:SW_MX_1u, symbol Switch:SW_Push
- SW1: footprint Button_Switch_THT:SW_NKK_GW12LJP -> PCM_marbastlib-mx:SW_MX_1u
- SW10: renamed from SW50; footprint Button_Switch_THT:SW_NKK_GW12LJP -> PCM_marbastlib-mx:SW_MX_1u
- SW11: renamed from SW49; footprint Button_Switch_THT:SW_NKK_GW12LJP -> PCM_marbastlib-mx:SW_MX_1u
- SW12: renamed from SW51; footprint Button_Switch_THT:SW_NKK_GW12LJP -> PCM_marbastlib-mx:SW_MX_1u
- SW13: renamed from SW3; footprint Button_Switch_THT:SW_NKK_GW12LJP -> PCM_marbastlib-mx:SW_MX_1u
- SW14: renamed from SW18; footprint Button_Switch_THT:SW_NKK_GW12LJP -> PCM_marbastlib-mx:SW_MX_1u
- SW15: renamed from SW34; footprint Button_Switch_THT:SW_NKK_GW12LJP -> PCM_marbastlib-mx:SW_MX_1u
- SW16: renamed from SW53; footprint Button_Switch_THT:SW_NKK_GW12LJP -> PCM_marbastlib-mx:SW_MX_1u
- SW17: renamed from SW52; footprint Button_Switch_THT:SW_NKK_GW12LJP -> PCM_marbastlib-mx:SW_MX_1u
- SW18: renamed from SW54; footprint Button_Switch_THT:SW_NKK_GW12LJP -> PCM_marbastlib-mx:SW_MX_1u
- SW19: renamed from SW4; footprint Button_Switch_THT:SW_NKK_GW12LJP -> PCM_marbastlib-mx:SW_MX_1u
- SW2: renamed from SW16; footprint Button_Switch_THT:SW_NKK_GW12LJP -> PCM_marbastlib-mx:SW_MX_1u
- SW20: renamed from SW19; footprint Button_Switch_THT:SW_NKK_GW12LJP -> PCM_marbastlib-mx:SW_MX_1u
- SW21: renamed from SW35; footprint Button_Switch_THT:SW_NKK_GW12LJP -> PCM_marbastlib-mx:SW_MX_1u
- SW22: renamed from SW56; footprint Button_Switch_THT:SW_NKK_GW12LJP -> PCM_marbastlib-mx:SW_MX_1u
- SW23: renamed from SW55; footprint Button_Switch_THT:SW_NKK_GW12LJP -> PCM_marbastlib-mx:SW_MX_1u
- SW24: renamed from SW36; footprint Button_Switch_THT:SW_NKK_GW12LJP -> PCM_marbastlib-mx:SW_MX_1u
- SW25: renamed from SW5; footprint Button_Switch_THT:SW_NKK_GW12LJP -> PCM_marbastlib-mx:SW_MX_1u
- SW26: renamed from SW20; footprint Button_Switch_THT:SW_NKK_GW12LJP -> PCM_marbastlib-mx:SW_MX_1u
- SW27: renamed from SW59; footprint Button_Switch_THT:SW_NKK_GW12LJP -> PCM_marbastlib-mx:SW_MX_1u
- SW28: renamed from SW58; footprint Button_Switch_THT:SW_NKK_GW12LJP -> PCM_marbastlib-mx:SW_MX_1u
- SW29: renamed from SW6; footprint Button_Switch_THT:SW_NKK_GW12LJP -> PCM_marbastlib-mx:SW_MX_1u
- SW3: renamed from SW31; footprint Button_Switch_THT:SW_NKK_GW12LJP -> PCM_marbastlib-mx:SW_MX_1u
- SW30: renamed from SW21; footprint Button_Switch_THT:SW_NKK_GW12LJP -> PCM_marbastlib-mx:SW_MX_1u
- SW31: renamed from SW37; footprint Button_Switch_THT:SW_NKK_GW12LJP -> PCM_marbastlib-mx:SW_MX_1u
- SW32: renamed from SW62; footprint Button_Switch_THT:SW_NKK_GW12LJP -> PCM_marbastlib-mx:SW_MX_1u
- SW33: renamed from SW61; footprint Button_Switch_THT:SW_NKK_GW12LJP -> PCM_marbastlib-mx:SW_MX_1u
- SW34: renamed from SW63; footprint Button_Switch_THT:SW_NKK_GW12LJP -> PCM_marbastlib-mx:SW_MX_1u
- SW35: renamed from SW7; footprint Button_Switch_THT:SW_NKK_GW12LJP -> PCM_marbastlib-mx:SW_MX_1u
- SW36: renamed from SW22; footprint Button_Switch_THT:SW_NKK_GW12LJP -> PCM_marbastlib-mx:SW_MX_1u
- SW37: renamed from SW38; footprint Button_Switch_THT:SW_NKK_GW12LJP -> PCM_marbastlib-mx:SW_MX_1u
- SW38: renamed from SW65; footprint Button_Switch_THT:SW_NKK_GW12LJP -> PCM_marbastlib-mx:SW_MX_1u
- SW39: renamed from SW64; footprint Button_Switch_THT:SW_NKK_GW12LJP -> PCM_marbastlib-mx:SW_MX_1u
- SW4: renamed from SW47; footprint Button_Switch_THT:SW_NKK_GW12LJP -> PCM_marbastlib-mx:SW_MX_1u
- SW40: renamed from SW8; footprint Button_Switch_THT:SW_NKK_GW12LJP -> PCM_marbastlib-mx:SW_MX_1u
- SW41: renamed from SW23; footprint Button_Switch_THT:SW_NKK_GW12LJP -> PCM_marbastlib-mx:SW_MX_1u
- SW42: renamed from SW39; footprint Button_Switch_THT:SW_NKK_GW12LJP -> PCM_marbastlib-mx:SW_MX_1u
- SW43: renamed from SW68; footprint Button_Switch_THT:SW_NKK_GW12LJP -> PCM_marbastlib-mx:SW_MX_1u
- SW44: renamed from SW67; footprint Button_Switch_THT:SW_NKK_GW12LJP -> PCM_marbastlib-mx:SW_MX_1u
- SW45: renamed from SW9; footprint Button_Switch_THT:SW_NKK_GW12LJP -> PCM_marbastlib-mx:SW_MX_1u
- SW46: renamed from SW24; footprint Button_Switch_THT:SW_NKK_GW12LJP -> PCM_marbastlib-mx:SW_MX_1u
- SW47: renamed from SW40; footprint Button_Switch_THT:SW_NKK_GW12LJP -> PCM_marbastlib-mx:SW_MX_1u
- SW48: renamed from SW71; footprint Button_Switch_THT:SW_NKK_GW12LJP -> PCM_marbastlib-mx:SW_MX_1u
- SW49: renamed from SW70; footprint Button_Switch_THT:SW_NKK_GW12LJP -> PCM_marbastlib-mx:SW_MX_1u
- SW5: renamed from SW46; footprint Button_Switch_THT:SW_NKK_GW12LJP -> PCM_marbastlib-mx:SW_MX_1u
- SW50: renamed from SW72; footprint Button_Switch_THT:SW_NKK_GW12LJP -> PCM_marbastlib-mx:SW_MX_1u
- SW51: renamed from SW10; footprint Button_Switch_THT:SW_NKK_GW12LJP -> PCM_marbastlib-mx:SW_MX_1u
- SW52: renamed from SW25; footprint Button_Switch_THT:SW_NKK_GW12LJP -> PCM_marbastlib-mx:SW_MX_1u
- SW53: renamed from SW42; footprint Button_Switch_THT:SW_NKK_GW12LJP -> PCM_marbastlib-mx:SW_MX_1u
- SW54: renamed from SW74; footprint Button_Switch_THT:SW_NKK_GW12LJP -> PCM_marbastlib-mx:SW_MX_1u
- SW55: renamed from SW73; footprint Button_Switch_THT:SW_NKK_GW12LJP -> PCM_marbastlib-mx:SW_MX_1u
- SW56: renamed from SW75; footprint Button_Switch_THT:SW_NKK_GW12LJP -> PCM_marbastlib-mx:SW_MX_1u
- SW58: renamed from SW11; footprint Button_Switch_THT:SW_NKK_GW12LJP -> PCM_marbastlib-mx:SW_MX_1u
- SW59: renamed from SW27; footprint Button_Switch_THT:SW_NKK_GW12LJP -> PCM_marbastlib-mx:SW_MX_1u
- SW6: renamed from SW48; footprint Button_Switch_THT:SW_NKK_GW12LJP -> PCM_marbastlib-mx:SW_MX_1u
- SW61: renamed from SW77; footprint Button_Switch_THT:SW_NKK_GW12LJP -> PCM_marbastlib-mx:SW_MX_1u
- SW62: renamed from SW78; footprint Button_Switch_THT:SW_NKK_GW12LJP -> PCM_marbastlib-mx:SW_MX_1u
- SW63: renamed from SW12; footprint Button_Switch_THT:SW_NKK_GW12LJP -> PCM_marbastlib-mx:SW_MX_1u
- SW67: renamed from SW79; footprint Button_Switch_THT:SW_NKK_GW12LJP -> PCM_marbastlib-mx:SW_MX_1u
- SW68: renamed from SW81; footprint Button_Switch_THT:SW_NKK_GW12LJP -> PCM_marbastlib-mx:SW_MX_1u
- SW7: renamed from SW2; footprint Button_Switch_THT:SW_NKK_GW12LJP -> PCM_marbastlib-mx:SW_MX_1u
- SW76: renamed from SW13; footprint Button_Switch_THT:SW_NKK_GW12LJP -> PCM_marbastlib-mx:SW_MX_1u
- SW77: renamed from SW28; footprint Button_Switch_THT:SW_NKK_GW12LJP -> PCM_marbastlib-mx:SW_MX_1u
- SW78: renamed from SW43; footprint Button_Switch_THT:SW_NKK_GW12LJP -> PCM_marbastlib-mx:SW_MX_1u
- SW79: renamed from SW84; footprint Button_Switch_THT:SW_NKK_GW12LJP -> PCM_marbastlib-mx:SW_MX_1u
- SW8: renamed from SW17; footprint Button_Switch_THT:SW_NKK_GW12LJP -> PCM_marbastlib-mx:SW_MX_1u
- SW80: renamed from SW14; footprint Button_Switch_THT:SW_NKK_GW12LJP -> PCM_marbastlib-mx:SW_MX_1u
- SW81: renamed from SW29; footprint Button_Switch_THT:SW_NKK_GW12LJP -> PCM_marbastlib-mx:SW_MX_1u
- SW82: renamed from SW44; footprint Button_Switch_THT:SW_NKK_GW12LJP -> PCM_marbastlib-mx:SW_MX_1u
- SW83: renamed from SW85; footprint Button_Switch_THT:SW_NKK_GW12LJP -> PCM_marbastlib-mx:SW_MX_1u
- SW84: renamed from SW87; footprint Button_Switch_THT:SW_NKK_GW12LJP -> PCM_marbastlib-mx:SW_MX_1u
- SW85: renamed from SW15; footprint Button_Switch_THT:SW_NKK_GW12LJP -> PCM_marbastlib-mx:SW_MX_1u
- SW86: renamed from SW30; footprint Button_Switch_THT:SW_NKK_GW12LJP -> PCM_marbastlib-mx:SW_MX_1u
- SW87: renamed from SW45; footprint Button_Switch_THT:SW_NKK_GW12LJP -> PCM_marbastlib-mx:SW_MX_1u
- SW88: renamed from SW90; footprint Button_Switch_THT:SW_NKK_GW12LJP -> PCM_marbastlib-mx:SW_MX_1u
- SW9: renamed from SW33; footprint Button_Switch_THT:SW_NKK_GW12LJP -> PCM_marbastlib-mx:SW_MX_1u
- renumbered D50 to D10, D49 to D11, D51 to D12, D3 to D13, D18 to D14, D34 to D15, D53 to D16, D52 to D17, D54 to D18, D4 to D19, D16 to D2, D19 to D20, D35 to D21, D56 to D22, D55 to D23, D36 to D24, D5 to D25, D20 to D26, D59 to D27, D58 to D28, D6 to D29, D31 to D3, D21 to D30, D37 to D31, D62 to D32, D61 to D33, D63 to D34, D7 to D35, D22 to D36, D38 to D37, D65 to D38, D64 to D39, D47 to D4, D8 to D40, D23 to D41, D39 to D42, D68 to D43, D67 to D44, D9 to D45, D24 to D46, D40 to D47, D71 to D48, D70 to D49, D46 to D5, D72 to D50, D10 to D51, D25 to D52, D42 to D53, D74 to D54, D73 to D55, D75 to D56, D11 to D57, D27 to D58, D48 to D6, D77 to D60, D78 to D61, D12 to D62, D79 to D66, D81 to D67, D2 to D7, D13 to D75, D28 to D76, D43 to D77, D84 to D78, D14 to D79, D17 to D8, D29 to D80, D44 to D81, D85 to D82, D87 to D83, D15 to D84, D30 to D85, D45 to D86, D90 to D87, D33 to D9
Connections:
- net COLUAN14: no longer SW85.1, SW86.1, SW87.1
- net COLUNA1: now also SW9.1
- net COLUNA10: now also SW59.1, SW57.1, SW60.1
- net COLUNA11: now also SW64.1, SW65.1, SW66.1; no longer SW53.1, SW59.1
- net COLUNA12: now also SW70.1, SW71.1, SW72.1, SW73.1; no longer SW76.1, SW77.1, SW78.1
- net COLUNA13: now also SW76.1, SW74.1, SW75.1; no longer SW80.1, SW81.1, SW82.1
- net COLUNA2: now also SW15.1; no longer SW9.1
- net COLUNA3: now also SW21.1; no longer SW15.1
- net COLUNA4: now also SW24.1; no longer SW21.1
- net COLUNA5: now also SW31.1; no longer SW24.1
- net COLUNA6: now also SW37.1; no longer SW31.1
- net COLUNA7: now also SW42.1; no longer SW37.1
- net COLUNA8: now also SW47.1; no longer SW42.1
- net COLUNA9: now also SW53.1; no longer SW47.1
- net LINHA0: now also D68.1 (K)
- net LINHA1: now also D63.1 (K), D69.1 (K), D73.1 (K)
- net LINHA2: now also D59.1 (K), D64.1 (K), D70.1 (K), D74.1 (K)
- net LINHA3: now also D65.1 (K), D71.1 (K)
- net LINHA4: now also D72.1 (K), SW57.2
- net COLUAN15: now reaches A1.20 (GPIO15)
- net COLUAN15: now also SW85.1
- net COLUAN16: now reaches A1.29 (GPIO22)
- net COLUAN16: now also SW86.1, SW87.1
- new net: D63.2 (A), SW64.2
- new net: D68.2 (A), SW69.2
- new net: D69.2 (A), SW70.2
- new net: D70.2 (A), SW71.2
- new net: D59.2 (A), SW60.2
- new net: D73.2 (A), SW74.2
- new net: D64.2 (A), SW65.2
- new net: D71.2 (A), SW72.2
- new net: D65.2 (A), SW66.2
- new net: D74.2 (A), SW75.2
- new net: D72.2 (A), SW73.2
- new net COLUAN12: SW69.1
- new net COLUNA14: SW77.1, SW78.1, SW80.1
- new net COLUNA15: SW81.1, SW82.1
- no-connect marks 13 -> 11
Other:
- moved on the sheet: D15, D21, D24, D31, D37, D42, D47, D53, D58, D75, D76, D77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
